Commit message: neuer LIDAR

File: catkin_ws/src/turtlebot3/turtlebot3_description/urdf/turtlebot3_waffle_pi.urdf.xacro (robot description, xacro)
@@ -282,7 +282,7 @@
   <link name="base_scan">
     <visual>
-      <origin xyz="0 0 0.05" rpy="0 0 0"/>
-      <geometry>
-        <mesh filename="package://turtlebot3_description/meshes/sensors/lds.stl" scale="0.001 0.001 0.001"/>
+      <origin xyz="0.014 0 0.05" rpy="0 0 0"/>
+      <geometry>
+        <mesh filename="package://turtlebot3_description/meshes/sensors/rplidar.stl" scale="0.001 0.001 0.001"/>
       </geometry>
       <material name="dark"/>

Commit message: Anpassungen SLAM

File: catkin_ws/src/turtlebot3/turtlebot3_description/urdf/turtlebot3_waffle_pi.urdf.xacro (robot description, xacro)
@@ -278,5 +278,5 @@
     <parent link="base_link"/>
     <child link="base_scan"/>
-    <origin xyz="0 0 -0.65" rpy="0 0 0"/>
+    <origin xyz="0 0 -0.65" rpy="3.14 3.14 0"/>
   </joint>
   <link name="base_scan">
